File: hardware/gpdi.kicad_sch (KiCad schematic)
At the start: 9 parts, among them J1 GPDI_A, Q1 BSN20

Commit message: Decoupled DDR3 and drew RJ45 connector
Parts:
- C15: LCSC Part # (none) -> C1525
- R16, R17: footprint Resistor_SMD:R_0402_1005Metric -> Resistor_SMD:R_0603_1608Metric; LCSC Part # (none) -> C22984
- R18, R19: footprint Resistor_SMD:R_0603_1608Metric -> Resistor_SMD:R_0402_1005Metric; LCSC Part # (none) -> C4109
Other:
- company: (none) -> Icy Electronics
- title: (none) -> Icepi CM0
Changed lines of the file:
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@@
 	(generator_version "9.0")
 	(paper "A4")
+	(title_block
+		(title "Icepi CM0")
+		(date "2025-11-03")
+		(rev "v1.0")
+		(company "Icy Electronics")
+		(comment 1 "Chengyin Yao (cheyao)")
+		(comment 2 "https://github.com/cheyao/icepi-cm0")
+	)
 	(bus_alias "GPDI"
 		(members "GPDI_D2+" "GPDI_D2-" "GPDI_D1+" "GPDI_D1-" "GPDI_D0+" "GPDI_D0-"
@@
 			)
 		)
-		(property "Footprint" "Resistor_SMD:R_0603_1608Metric"
+		(property "Footprint" "Resistor_SMD:R_0402_1005Metric"
 			(at 125.222 77.47 90)
 			(effects
@@
 			)
 		)
-		(property "LCSC Part #" ""
+		(property "LCSC Part #" "C4109"
 			(at 127 77.47 0)
 			(effects
@@
 			)
 		)
+		(property "LCSC Part #" "C1525"
+			(at 160.02 86.36 0)
+			(effects
+				(font
+					(size 1.27 1.27)
+				)
+				(hide yes)
+			)
+		)
 		(pin "1"
 		)
@@
 			)
 		)
-		(property "Footprint" "Resistor_SMD:R_0402_1005Metric"
+		(property "Footprint" "Resistor_SMD:R_0603_1608Metric"
 			(at 149.352 46.99 90)
 			(effects
@@
 		(property "Description" "Resistor"
 			(at 151.13 46.99 0)
+			(effects
+				(font
+					(size 1.27 1.27)
+				)
+				(hide yes)
+			)
+		)
+		(property "LCSC Part #" "C22984"
+			(at 151.13 46.99 90)
 			(effects
 				(font
@@
 			)
 		)
-		(property "Footprint" "Resistor_SMD:R_0603_1608Metric"
+		(property "Footprint" "Resistor_SMD:R_0402_1005Metric"
 			(at 130.302 77.47 90)
 			(effects
@@
 			)
 		)
-		(property "LCSC Part #" ""
+		(property "LCSC Part #" "C4109"
 			(at 132.08 77.47 0)
 			(effects
@@
 			)
 		)
-		(property "Footprint" "Resistor_SMD:R_0402_1005Metric"
+		(property "Footprint" "Resistor_SMD:R_0603_1608Metric"
 			(at 135.382 46.99 90)
 			(effects
@@
 			(effects
 				(font
+					(size 1.27 1.27)
+				)
+				(hide yes)
+			)
+		)
+		(property "LCSC Part #" "C22984"
+			(at 137.16 46.99 90)
+			(effects
+				(font
