File: hardware/cm0.kicad_pcb (KiCad board)
At the start: 4 copper layers, 100 x 90 mm, 116 parts, among them J1 GPDI_A, J2 USB_C_Receptacle_USB2.0_14P, J3 USB_C_Receptacle_USB2.0_14P, J4 USB_A_Stacked, J5 USB_C_Receptacle_USB2.0_14P, J6 AIPEX-1, J7 Micro_SD_Card_Det1, J8 RJ45_Hanrun_HR913550A_Horizon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, Q1 BSN20, U1 H3, U10 TPD2EUSB30, U11 SY6280AAC, U12 HUSB237, U13 AW13412HDNR, U14 UCL0524P, U15 UCL0524P, U16 EMMC5.1_BGA153, U2 H5TQ4G63EFR, U3 AP6212, U4 SY6280AAC, U5 SY6280AAC, U6 TPD2EUSB30, U7 TPD2EUSB30, U8 SY6280AAC, U9 TPD2EUSB30, Y1 26MHz

Commit message: Initial layout
Parts:
- removed the C45 at (93.7, 70.1)
- removed the J6 at (98.9, 65.1)
- removed JP1: RF_BK, Jumper:SolderJumper-2_P1.3mm_Bridged_RoundedPad1.0x1.5mm
- removed the R31 at (111.7, 94.1)
- removed TP1: 3V3, TestPoint:TestPoint_Pad_D1.0mm
- removed the U13 at (92.0, 69.5)
- added C50: 10uF, Capacitor_SMD:C_0603_1608Metric, F.Cu at (142.1, 91.7)
- added C51: 10uF, Capacitor_SMD:C_0603_1608Metric, F.Cu at (142.1, 94.2)
- added J10: AudioJack_PJ-342, cm0:Jack_3.5mm_SHOUHAN_PJ-342, F.Cu at (136.0, 100.6)
- added J8: Conn_02x20_Odd_Even, Connector_PinHeader_2.54mm:PinHeader_2x20_P2.54mm_Vertical, F.Cu at (136.4, 89.1)
- added J9: Conn_01x03, Connector_PinHeader_2.54mm:PinHeader_1x03_P2.54mm_Vertical, F.Cu at (97.1, 125.0)
- added Q2: BSN20, Package_TO_SOT_SMD:SOT-23, F.Cu at (103.0, 120.2)
- added R34: 10k, Resistor_SMD:R_0402_1005Metric, F.Cu at (100.9, 111.2)
- added R35: 33, Resistor_SMD:R_0402_1005Metric, F.Cu at (97.8, 121.2)
- added R36: 33, Resistor_SMD:R_0402_1005Metric, F.Cu at (99.8, 121.2)
- added R37: 10k, Resistor_SMD:R_0402_1005Metric, F.Cu at (95.8, 121.2)
- added U15: EMMC5.1_BGA153, Package_BGA:LFBGA-153_11.5x13mm_Layout14x14_P0.5mm, F.Cu at (98.8, 101.6)
- AE1: value PCB_Antenna -> 2450AT18A100E; footprint RF_Antenna:Texas_SWRA117D_2.4GHz_Left -> RF_Antenna:Johanson_2450AT18x100
- C25: renamed from C37; moved to B.Cu
- C26: renamed from C41; moved to B.Cu
- C27: renamed from C44; moved to B.Cu
- C29: renamed from C43; moved to B.Cu
- C3: renamed from C14; moved to B.Cu
- C4: renamed from C13; moved to B.Cu
- C47: value 1nF -> 1uF
- C48: value 1uF -> NC
- C49: value 100nF -> NC
- J3: renamed from J5; footprint Connector_USB:USB_C_Receptacle_HRO_TYPE-C-31-M-12 -> cm0:USB_C_Receptacle_HRO_TYPE-C-31-M-12
- J4: renamed from J2; footprint Connector_USB:USB_C_Receptacle_HRO_TYPE-C-31-M-12 -> cm0:USB_C_Receptacle_HRO_TYPE-C-31-M-12
- J5: renamed from J3; footprint Connector_USB:USB_C_Receptacle_HRO_TYPE-C-31-M-12 -> cm0:USB_C_Receptacle_HRO_TYPE-C-31-M-12
- R1, R2: value 22 -> 33; moved to F.Cu
- R10: renamed from R9; value 30k -> 33k; footprint Resistor_SMD:R_0603_1608Metric -> Resistor_SMD:R_0402_1005Metric
- R11: renamed from R10; value 30k -> 33k; footprint Resistor_SMD:R_0603_1608Metric -> Resistor_SMD:R_0402_1005Metric
- R12: renamed from R11; value 30k -> 33k; footprint Resistor_SMD:R_0603_1608Metric -> Resistor_SMD:R_0402_1005Metric
- R13: renamed from R12; value 30k -> 33k; footprint Resistor_SMD:R_0603_1608Metric -> Resistor_SMD:R_0402_1005Metric
- R15: renamed from R14; value 22 -> 33
- R21: renamed from R16; value 30k -> 33k; footprint Resistor_SMD:R_0603_1608Metric -> Resistor_SMD:R_0402_1005Metric
- R22: renamed from R17; value 30k -> 33k; footprint Resistor_SMD:R_0603_1608Metric -> Resistor_SMD:R_0402_1005Metric
- R23: renamed from R24; moved to B.Cu
- R24: renamed from R25; moved to B.Cu
- R33: renamed from R32; value 22 -> 33
- R9: renamed from R8; value 30k -> 33k; footprint Resistor_SMD:R_0603_1608Metric -> Resistor_SMD:R_0402_1005Metric
- U16: value EMMC5.1_BGA153 -> TPD2EUSB30; footprint Package_BGA:LFBGA-153_11.5x13mm_Layout14x14_P0.5mm -> Package_TO_SOT_SMD:Texas_DRT-3
- moved C27 85.8 mm to (69.6, 99.8)
- moved C29 84.5 mm to (69.6, 94.2)
- moved AE1 80.2 mm to (65.2, 139.4), turned to -90 degrees
- moved R17 72.0 mm to (70.0, 106.3)
- moved R24 71.7 mm to (124.5, 136.5), turned to 180 degrees
- moved C32 71.4 mm to (69.7, 140.2), turned to 180 degrees
- moved Y1 69.9 mm to (69.7, 138.3), turned to 90 degrees
- moved J3 68.7 mm to (97.3, 140.9), turned to 0 degrees
- moved C33 68.4 mm to (69.7, 136.3), turned to 0 degrees
- moved C35 67.5 mm to (139.2, 148.1), turned to 0 degrees
- moved D2 66.9 mm to (139.2, 150.2), turned to -90 degrees
- moved J4 66.3 mm to (122.3, 140.9), turned to 0 degrees
- moved C28 65.9 mm to (71.7, 136.2), turned to 90 degrees
- moved R20 65.2 mm to (134.4, 152.1), turned to 180 degrees
- moved J1 64.2 mm to (80.4, 92.6), turned to -90 degrees
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- renumbered C5 to C10, C39 to C11, C26 to C12, C27 to C13, C28 to C14, C33 to C15, C40 to C16, C38 to C17, C29 to C18, C36 to C19, C30 to C20, C34 to C21, C31 to C22, C35 to C23, C6 to C24, C7 to C28, C8 to C30, C9 to C31, C10 to C32, C11 to C33, C12 to C34, C15 to C35, C25 to C36, C21 to C37, C23 to C38, C22 to C39, C24 to C40, C20 to C41, C19 to C42, C17 to C43, C18 to C44, C50 to C45, C3 to C5, C16 to C6, C32 to C7, C42 to C8, C4 to C9, D2 to D1, D1 to D2, J8 to J1, J1 to J2, J4 to J6, R13 to R14, R15 to R16, R30 to R17, R28 to R18, R18 to R20, R22 to R25, R23 to R26, R26 to R27, R29 to R28, R20 to R29, R21 to R30, R33 to R31, R34 to R32, R27 to R4, R4 to R5, R5 to R6, R6 to R7, R7 to R8, U6 to U11, U7 to U12, U4 to U13, U5 to U14, U14 to U4, U15 to U5, U12 to U6, U8 to U7, U11 to U8
Connections:
- C31 pad 2: Net-(U13-ANT) -> Net-(AE1-A)
- C46 pad 1: +3V3 -> Net-(U15-VDDI)
- C47 pad 1: +3V3 -> GND
- C47 pad 2: GND -> Net-(U15-VDDI)
- C48 pad 1: GND -> Net-(U3-WL_BT_ANT)
- C48 pad 2: Net-(U16-VDDI) -> GND
- C49 pad 1: Net-(U16-VDDI) -> Net-(AE1-A)
- J2 pad 12: /GPDI/GPDI_GCLK- -> /GPDI/GPDI_CLK-
- R1 pad 1: /DDR3/CLK+ -> Net-(J10-Pad3)
- R1 pad 2: /H3/C+ -> Net-(C50-Pad1)
- R2 pad 1: /H3/C- -> Net-(J10-Pad4)
- R2 pad 2: /DDR3/CLK- -> Net-(C51-Pad1)
- U1 pad A1: (no net) -> unconnected-(U1G-JTAG-SEL0-PadA1)
- U1 pad AA19: /H3/C+ -> /DDR3/CLK+
- U1 pad AA2: (no net) -> unconnected-(U1H-MICIN2N-PadAA2)
- U1 pad AA20: /H3/C- -> /DDR3/CLK-
- U1 pad AA3: (no net) -> /H3/AUDIO_L
- U1 pad AA5: (no net) -> unconnected-(U1G-KEYADC-PadAA5)
- U1 pad AA6: (no net) -> unconnected-(U1G-NMI-PadAA6)
- U1 pad B2: (no net) -> unconnected-(U1G-JTAG-SEL1-PadB2)
- U1 pad C8: (no net) -> unconnected-(U1F-PE7-PadC8)
- U1 pad D1: unconnected-(U1C-PG12-PadD1) -> /H3/BT_HOST_WAKE
- U1 pad D2: unconnected-(U1C-PG11-PadD2) -> /H3/~{BT_RST}
- U1 pad F10: (no net) -> /H3/TV_OUT
- U1 pad F5: unconnected-(U1F-PA4-PadF5) -> /H3/CPU_TX
- U1 pad G9: (no net) -> unconnected-(U1D-V33_TV-PadG9)
- U1 pad H6: unconnected-(U1F-PA5-PadH6) -> /H3/CPU_RX
- U1 pad H8: (no net) -> unconnected-(U1D-GND_TV-PadH8)
- U1 pad K1: (no net) -> unconnected-(U1G-X24MOUT-PadK1)
- U1 pad K2: (no net) -> unconnected-(U1G-X24MIN-PadK2)
- U1 pad K6: (no net) -> unconnected-(U1G-VCC_RTC-PadK6)
- U1 pad L5: (no net) -> unconnected-(U1G-PLLTEST-PadL5)
- U1 pad M3: unconnected-(U1C-PG10-PadM3) -> /H3/BT_WAKE
- U1 pad M4: (no net) -> unconnected-(U1G-RTC_VIO-PadM4)
- U1 pad N3: (no net) -> unconnected-(U1G-VCC_PLL-PadN3)
- U1 pad P3: (no net) -> /H3/WIFI_32K
- U1 pad T10: (no net) -> unconnected-(U1B-VDD-CPUFB-PadT10)
- U1 pad T5: (no net) -> unconnected-(U1G-TEST-PadT5)
- U1 pad T9: (no net) -> GND
- U1 pad U3: (no net) -> unconnected-(U1H-AGND-PadU3)
- U1 pad U4: (no net) -> unconnected-(U1G-X32KOUT-PadU4)
- U1 pad V1: (no net) -> unconnected-(U1H-LINEINL-PadV1)
- U1 pad V3: (no net) -> unconnected-(U1H-AVCC-PadV3)
- U1 pad V4: (no net) -> unconnected-(U1H-VRP-PadV4)
- U1 pad V5: (no net) -> unconnected-(U1G-X32KIN-PadV5)
- U1 pad V6: (no net) -> unconnected-(U1G-RESET-PadV6)
- U1 pad W1: (no net) -> unconnected-(U1H-LINEINR-PadW1)
- U1 pad W2: (no net) -> unconnected-(U1H-MICIN1P-PadW2)
- U1 pad W3: (no net) -> unconnected-(U1H-MBIAS-PadW3)
- U1 pad W5: (no net) -> unconnected-(U1H-VRA2-PadW5)
- U1 pad W6: (no net) -> unconnected-(U1G-UBOOT-PadW6)
- U1 pad Y1: (no net) -> unconnected-(U1H-MICIN1N-PadY1)
- U1 pad Y2: (no net) -> unconnected-(U1H-MICIN2P-PadY2)
- U1 pad Y3: (no net) -> /H3/AUDIO_R
- U1 pad Y4: (no net) -> unconnected-(U1H-VRA1-PadY4)
- U5 pad 5: /GPDI/GPDI_GCLK- -> /GPDI/GPDI_CLK-
- U5 pad 6: /GPDI/GPDI_GCLK- -> /GPDI/GPDI_CLK-
Routing:
- net /GPDI/GPDI_CLK-: track 1.89 -> 32.1 mm
- net /GPDI/GPDI_CLK+: track 1.89 -> 31.7 mm
- net /H3/USB_D0-: track 0.00 -> 28.7 mm
- net /H3/USB_D0+: track 0.00 -> 28.5 mm
- net /GPDI/GPDI_D0-: track 1.16 -> 29.6 mm
- net /GPDI/GPDI_D0+: track 1.16 -> 29.1 mm
- net /GPDI/GPDI_D1-: track 1.95 -> 28.5 mm
- net /GPDI/GPDI_D1+: track 1.95 -> 27.9 mm
- net /GPDI/GPDI_D2-: track 1.68 -> 26.9 mm
- net /GPDI/GPDI_D2+: track 0.76 -> 25.7 mm
- net /H3/USB_D1-: track 0.00 -> 21.9 mm
- net /H3/USB_D1+: track 0.00 -> 21.1 mm
- net /DDR3/CLK+: track 19.6 -> 24.9 mm, vias 1 -> 2
- net /DDR3/CLK-: track 19.6 -> 24.9 mm, vias 1 -> 2
- net /H3/C+: track 4.28 -> 0.00 mm, vias 1 -> 0
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Other:
- board size 100 x 90 mm -> 85 x 60 mm
