File: hardware/cm0.kicad_sch (KiCad schematic)
At the start: 0 parts

Commit message: Initial layout
Other:
- added sheet Audio (audio.kicad_sch)
Changed lines of the file:
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@@
+	)
+	(sheet
+		(at 143.764 59.69)
+		(size 22.606 15.24)
+		(exclude_from_sim no)
+		(in_bom yes)
+		(on_board yes)
+		(dnp no)
+		(fields_autoplaced yes)
+		(stroke
+			(width 0.1524)
+			(type solid)
+		)
+		(fill
+			(color 0 0 0 0.0000)
+		)
+		(property "Sheetname" "Audio"
+			(at 143.764 58.9784 0)
+			(effects
+				(font
+					(size 1.27 1.27)
+				)
+				(justify left bottom)
+			)
+		)
+		(property "Sheetfile" "audio.kicad_sch"
+			(at 143.764 75.5146 0)
+			(effects
+				(font
+					(size 1.27 1.27)
+				)
+				(justify left top)
+			)
+		)
+		(instances
+			(project "cm0"
+				(path "/b53f5dbb-8078-4818-9e8f-fdf90ba6d854"
+					(page "10")
+				)
+			)
+		)
 	)
 	(sheet
