File: hardware/wifi.kicad_sch (KiCad schematic)
At the start: 34 parts, among them J6 AIPEX-1, J8 RJ45_Hanrun_HR913550A_Horizon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, U13 AW13412HDNR, U3 AP6212, Y1 26MHz

Commit message: Initial layout
Parts:
- removed C45: 10pF, Capacitor_SMD:C_0402_1005Metric, symbol Device:C
- removed C46: 100nF, Capacitor_SMD:C_0402_1005Metric, symbol Device:C
- removed C47: 1nF, Capacitor_SMD:C_0402_1005Metric, symbol Device:C
- removed J6: AIPEX-1, Connector_Coaxial:U.FL_Hirose_U.FL-R-SMT-1_Vertical, symbol Connector:Conn_Coaxial_Small
- removed JP1: RF_BK, Jumper:SolderJumper-2_P1.3mm_Bridged_RoundedPad1.0x1.5mm, symbol Jumper:SolderJumper_2_Bridged
- removed TP1: 3V3, TestPoint:TestPoint_Pad_D1.0mm, symbol Connector:TestPoint
- removed U13: AW13412HDNR, cm0:DFN-6_1.1x0.7mm_P0.4mm, symbol cm0:AW13412HDNR
- added C48, C49: NC, Capacitor_SMD:C_0402_1005Metric, symbol Device:C
- AE1: value PCB_Antenna -> 2450AT18A100E; footprint RF_Antenna:Texas_SWRA117D_2.4GHz_Left -> RF_Antenna:Johanson_2450AT18x100; LCSC Part # (none) -> C89334; now in the parts list
- R10: renamed from R9; value 30k -> 33k; footprint Resistor_SMD:R_0603_1608Metric -> Resistor_SMD:R_0402_1005Metric; LCSC Part # C22984 -> C25779
- R11: renamed from R10; value 30k -> 33k; footprint Resistor_SMD:R_0603_1608Metric -> Resistor_SMD:R_0402_1005Metric; LCSC Part # C22984 -> C25779
- R12: renamed from R11; value 30k -> 33k; footprint Resistor_SMD:R_0603_1608Metric -> Resistor_SMD:R_0402_1005Metric; LCSC Part # C22984 -> C25779
- R13: renamed from R12; value 30k -> 33k; footprint Resistor_SMD:R_0603_1608Metric -> Resistor_SMD:R_0402_1005Metric; LCSC Part # C22984 -> C25779
- R15: renamed from R14; value 22 -> 33; LCSC Part # C25092 -> (none)
- R9: renamed from R8; value 30k -> 33k; footprint Resistor_SMD:R_0603_1608Metric -> Resistor_SMD:R_0402_1005Metric; LCSC Part # C22984 -> C25779
- renumbered C6 to C24, C37 to C25, C41 to C26, C44 to C27, C7 to C28, C43 to C29, C8 to C30, C9 to C31, C10 to C32, C11 to C33, C12 to C34, J8 to J1, R13 to R14, R15 to R16, R30 to R17, R28 to R18, R7 to R8
Connections:
- net GND: now also C48.2, C49.2
- net at AE1.1 (A): now also C31.2, C49.1
- net at C31.1, U3.2 (WL_BT_ANT): now also C48.1
Other:
- note removed: "Cut and solder to 3V3 for external antenna"
- moved on the sheet: AE1, C25, C26, C27, C29, C31, J1, R17, R18
