File: hardware/power_tree.kicad_sch (KiCad schematic)
At the start: 0 parts

Commit message: Decoupling on PCB side almost done
Other:
- note added: "3.3V/0.5A"
- note removed: "3.3V/2A"
Changed lines of the file:
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@@
 		)
 	)
-	(text "3.3V/2A"
+	(text "3.3V/1A"
 		(exclude_from_sim no)
 		(at 142.494 105.156 0)
@@
 	(text "H3 Debugging Guide"
 		(exclude_from_sim no)
-		(at 48.006 16.764 0)
+		(at 24.892 52.07 0)
 		(effects
 			(font
@@
 		)
 	)
-	(text "3.3V/2A"
+	(text "3.3V/0.5A"
 		(exclude_from_sim no)
 		(at 142.494 117.856 0)
@@
 		)
 	)
-	(text_box "SY8089A"
+	(text_box "SY8088"
 		(exclude_from_sim no)
 		(at 127 101.6 0)
@@
 		(exclude_from_sim no)
 		(at 15.24 15.24 0)
-		(size 20.32 20.32)
+		(size 29.21 20.32)
 		(margins 0.9525 0.9525 0.9525 0.9525)
 		(stroke
@@
 		)
 	)
-	(text_box "SY8089A"
+	(text_box "SY8088"
 		(exclude_from_sim no)
 		(at 127 114.3 0)
@@
 		)
 	)
-	(text_box "SY8088      1A\nSY8089A     2A\nSY8113B     3A"
+	(text_box "SY8088      1A   1.5MHz\nSY8089A     2A     1MHz\nSY8113B     3A   0.5MHz"
 		(exclude_from_sim no)
 		(at 15.24 40.64 0)
-		(size 20.574 7.62)
-		(margins 0.9525 0.9525 0.9525 0.9525)
-		(stroke
+		(size 29.21 7.62)
+		(margins 0.9525 0.9525 0.9525 0.9525)
+		(stroke
