File: hardware/cpu.kicad_sch (KiCad schematic)
At the start: 7 parts, among them U1 H3

Commit message: Finished DC DC converters and started decoupling the CPU
Parts:
- added C10, C11, C32: 4.7uF, Capacitor_SMD:C_0402_1005Metric, symbol Device:C
- added C12, C14, C18, C19, C23, C24, C26, C27, C29, C3, C31, C37, C38, C4, C5, C6, C7: 100nF, Capacitor_SMD:C_0402_1005Metric, symbol Device:C
- added C13, C16, C17, C21, C22, C25, C33, C35, C36: 1uF, Capacitor_SMD:C_0402_1005Metric, symbol Device:C
- added C15, C20, C28, C30: 10uF, Capacitor_SMD:C_0603_1608Metric, symbol Device:C
- added C34, C39: 15pF, Capacitor_SMD:C_0402_1005Metric, symbol Device:C
- added R3, R5: 0, Resistor_SMD:R_0402_1005Metric, symbol Device:R
- added R4: 220k, Resistor_SMD:R_0402_1005Metric, symbol Device:R
- added R6: 10M, Resistor_SMD:R_0402_1005Metric, symbol Device:R
- added R61: 47k, Resistor_SMD:R_0402_1005Metric, symbol Device:R
- added TP1: TestPoint, TestPoint:TestPoint_Pad_D1.0mm, symbol Connector:TestPoint
- added Y1: 32kHz, Crystal:Crystal_SMD_3215-2Pin_3.2x1.5mm, symbol Device:Crystal
- renumbered C2 to C1, C3 to C2, C4 to C8, C1 to C9, R4 to R1, R3 to R2
Connections:
- net +3V3 is gone; now on net +3V3_IO: C1.2, C2.2, C8.2, U1.G11 (VCC_USB), U1.H7 (VCC-PG), U1.J15 (VCC_PD), U1.J6 (GPDI_VCC)
- net VCC-IO is gone; now on net +3V3_IO: U1.G13 (VCC-IO), U1.G14 (VCC-IO), U1.G15 (VCC-IO), U1.H13 (VCC-IO), U1.H14 (VCC-IO), U1.J14 (VCC-IO)
- net VDD-CPUS is gone; now on net VDD_CPUS: U1.J7 (VDD-CPUS), U1.J8 (VDD-CPUS)
- net VDD-SYS is gone; now on net +1V2_SYSTEM: U1.H10 (VDD-SYS), U1.J10 (VDD-SYS), U1.J11 (VDD-SYS), U1.J12 (VDD-SYS), U1.K10 (VDD-SYS), U1.K11 (VDD-SYS), U1.K12 (VDD-SYS), U1.L10 (VDD-SYS), U1.L11 (VDD-SYS), U1.L12 (VDD-SYS), U1.L13 (VDD-SYS), U1.L14 (VDD-SYS)
- net +1V5: now also C35.2, C36.2, C37.2, C38.2
- net EPHY_LINK_LED: now also C6.2
- net EPHY_SPD_LED: now also C5.2
- net GND: now also U1.H8 (GND_TV), C10.2, C11.2, C12.1, C13.1, C14.1, C15.2, C16.1, C17.1, C18.1, C19.1, C20.2, C21.1, C22.1, C23.1, C24.1, C25.1, C26.1, C27.1, C3.1, C34.2, C35.1, C36.1, C37.1, C38.1, C39.2, C4.1, C5.1, C6.1, C7.1, R3.2, R5.2; no longer U1.T9 (GND-CPUFB)
- net AGND: now reaches U1.U3 (AGND)
- net AGND: now also C28.2, C29.1, C30.2, C31.1, C32.2, C33.1, R4.2, R5.1
- net +3V3_AVCC: now reaches U1.V3 (AVCC)
- net +3V3_AVCC: now also U1.G9 (V33_TV), U1.N3 (VCC_PLL), C12.2, C28.1, C29.2, C7.2
- net VRP: now reaches U1.V4 (VRP)
- net VRP: now also C30.1, C31.2
- net VRA2: now reaches U1.W5 (VRA2)
- net VRA2: now also C32.1, R4.1
- net VRA1: now reaches U1.Y4 (VRA1)
- net VRA1: now also C33.2
- net at U1.AA6 (NMI): now also R61.2
- net +3V3_RTC: now reaches U1.K6 (VCC_RTC)
- net +3V3_RTC: now also C27.2, R61.1
- net VDD_CPUS: now reaches U1.M4 (RTC_VIO)
- net VDD_CPUS: now also C11.1, C25.2, C26.2
- net X32KO: now reaches U1.U4 (X32KOUT)
- net X32KO: now also C39.1, R6.2, Y1.1
- net X32KI: now reaches U1.V5 (X32KIN)
- net X32KI: now also C34.1, R6.1, Y1.2
- net at U1.G10 (VDD-EFUSE): now also C10.1
- net +3V3_IO: now reaches U1.H11 (VDD-EFUSEEBP)
- net +3V3_IO: now also U1.G7 (EPHY_VCC), C13.2, C14.2, C3.2
- net PWR_VSET: now reaches U1.T4 (PL6)
- net +1V2_SYSTEM: now reaches U1.F8 (EPHY_VDD)
- net +1V2_SYSTEM: now also C20.1, C21.2, C22.2, C23.2, C24.2, C4.2
- net VDD-CPUX renamed +1V1_CPUX
- net +1V1_CPUX: now also C15.1, C16.2, C17.2, C18.2, C19.2
- new net: R3.1, U1.T9 (GND-CPUFB)
- new net PWR_CPUFB: TP1.1, U1.T10 (VDD-CPUFB)
- no-connect marks 9 -> 23
Other:
- moved on the sheet: C2, C8, R1, U1D, U1E, U1F, U1H

Commit message: Decoupling on PCB side almost done
Parts:
- removed C5, C6: 100nF, Capacitor_SMD:C_0402_1005Metric, symbol Device:C
- added C127, C128: 15pF, Capacitor_SMD:C_0402_1005Metric, symbol Device:C
- added C129: 4.7uF, Capacitor_SMD:C_0402_1005Metric, symbol Device:C
- added C130: 100nF, Capacitor_SMD:C_0402_1005Metric, symbol Device:C
- added Q5: MMBT3904, Package_TO_SOT_SMD:SOT-23, symbol Transistor_BJT:MMBT3904
- added R62: 100k, Resistor_SMD:R_0402_1005Metric, symbol Device:R
- added R63, R64, R65: 10k, Resistor_SMD:R_0402_1005Metric, symbol Device:R
- added R66, R67, R68: 47k, Resistor_SMD:R_0402_1005Metric, symbol Device:R
- added TP2, TP3: TestPoint, TestPoint:TestPoint_Pad_D1.0mm, symbol Connector:TestPoint
- added Y3: 24MHz, Crystal:Crystal_SMD_2016-4Pin_2.0x1.6mm, symbol Device:Crystal_GND24
- C10, C11, C32: LCSC Part # (none) -> C23733
- R3, R5: LCSC Part # (none) -> C17168
- R4: LCSC Part # (none) -> C25767
- R6: LCSC Part # (none) -> C26082
- R61: LCSC Part # (none) -> C25792
- TP1: now not fitted
Connections:
- net +3V3_AVCC: now also R62.1
- net +3V3_IO: now also C129.1, R67.1
- net +3V3_RTC: now also R65.1, R66.1, R68.1
- net GND: now also C127.2, C128.2, C130.1, Q5.2 (E), R63.2, Y3.1, Y3.3
- net at U1.A1 (JTAG-SEL0): now also TP2.1
- net KEYADC: now reaches U1.AA5 (KEYADC)
- net KEYADC: now also R62.2
- net at U1.B2 (JTAG-SEL1): now also TP3.1
- net X24MO: now reaches U1.K1 (X24MOUT)
- net X24MO: now also C128.1, Y3.4
- net X24MI: now reaches U1.K2 (X24MIN)
- net X24MI: now also C127.1, Y3.2
- net RESET: now reaches U1.V6 (RESET)
- net RESET: now also C130.2, Q5.3 (C), R65.2
- net UBOOT: now reaches U1.W6 (UBOOT)
- net UBOOT: now also R67.2
- net RECOVERY: now reaches U1.N2 (PL4)
- net RECOVERY: now also R68.2
- net PWR_KEY: now reaches U1.R1 (PL3)
- net PWR_KEY: now also R66.2
- new net: C129.2, R63.1, R64.1
- new net: Q5.1 (B), R64.2
- no-connect marks 23 -> 29
Other:
- note added: "Accessible via resistor"
- note added: "FIXME: KEYADC"
- note added: "This isn't a laptop so no power key & KEYADC"
- moved on the sheet: C1, C10, C11, C12, C13, C14, C15, C16, C17, C18, C19, C2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
